File: src-kicad/vumeter.sch (KiCad schematic (older format))
At the start: 35 parts, among them J1 JACK_TRS_5_PIN, J2 JACK_TRS_5_PIN, J3 Channel, J4 B2B_in, J5 B2B_out, J6 BARREL_JACK, J7 Switch, U1 LM358, U2 lm7805, U3 LM3915

Commit message: schematic modified 	now analyze stereo signal without lowpass and hipass filters.
Parts:
- removed 1n4007: D3, Diodes_ThroughHole:D_A-405_P10.16mm_Horizontal, symbol D
- removed C1: 10nF, Capacitors_ThroughHole:C_Rect_L7.0mm_W2.0mm_P5.00mm, symbol C
- removed C2: 100nF, Capacitors_ThroughHole:C_Rect_L7.0mm_W2.0mm_P5.00mm, symbol C
- removed J2: JACK_TRS_5_PIN, vumetro:Jack_TRS_3.5mm_5_pin, symbol JACK_TRS_5_PIN
- removed J3: Channel, Pin_Headers:Pin_Header_Straight_1x03_Pitch2.54mm, symbol CONN_01X03
- removed J4: B2B_in, Pin_Headers:Pin_Header_Straight_1x04_Pitch2.54mm, symbol CONN_01X04
- removed J5: B2B_out, Pin_Headers:Pin_Header_Straight_1x04_Pitch2.54mm, symbol CONN_01X04
- removed R3: 8k2, Resistors_ThroughHole:R_Axial_DIN0207_L6.3mm_D2.5mm_P2.54mm_Vertical, symbol R
- removed R4: 6k2, Resistors_ThroughHole:R_Axial_DIN0207_L6.3mm_D2.5mm_P2.54mm_Vertical, symbol R
- added C?: 10nF, Capacitors_ThroughHole:C_Rect_L7.0mm_W2.0mm_P5.00mm, symbol C
- added D?: 1n5822, Diodes_ThroughHole:D_A-405_P10.16mm_Horizontal, symbol D_Schottky
- added Dm? (x10): LED, LEDs:LED_D5.0mm, symbol LED-RESCUE-vumeter
- added R? (x3): 1k, Resistors_ThroughHole:R_Axial_DIN0207_L6.3mm_D2.5mm_P2.54mm_Vertical, symbol R
- added R?: 10k, Resistors_ThroughHole:R_Axial_DIN0207_L6.3mm_D2.5mm_P2.54mm_Vertical, symbol R
- added R?: 470k, Resistors_ThroughHole:R_Axial_DIN0207_L6.3mm_D2.5mm_P2.54mm_Vertical, symbol R
- added Rv?: 100k, Potentiometers:Potentiometer_Trimmer_ACP_CA9h2.5_Vertical_Px2.5mm_Py5.0mm, symbol POT-RESCUE-vumeter
- added U4: LM3915, Housings_DIP:DIP-18_W7.62mm_LongPads, symbol LM3915
- D1, Dm1, Dm10, Dm2, Dm3, Dm4, Dm5, Dm6, Dm7, Dm8, Dm9: symbol LED -> LED-RESCUE-vumeter
- Rv1: symbol POT -> POT-RESCUE-vumeter
Connections:
- net labels added: S_amp_left, S_amp_right
- net labels removed: S_amp, S_filtro
- wire segments 131 -> 165
- no-connect marks 5 -> 4
Other:
- note added: "Display - Left"
- note added: "Display - Right"
- note removed: "Board to board"
- note removed: "Display"
- note removed: "Filter"
- moved on the sheet: D1, J1, J6, J7, R1, R2, R8, Rv1, U1A, U2
